File: hardware/KungFuFlash.kicad_pcb (KiCad board)
At the start: 2 copper layers, 60.6 x 62 mm, 40 parts, among them J1 USB Power, J2 USB_B_Micro, J4 SWD, Q1 BC817, SW1 Reset, SW2 Menu, SW3 Special, U1 C64-Exp-Port, U2 AMS1117-3.3, U3 STM32F405RGTx, Y1 8MHz

Commit message: First try for SID file type, USB only mode and some helper files
Connections:
- net /R~W renamed /R~{W}
- net /~EXROM renamed /~{EXROM}
- net /~GAME renamed /~{GAME}
- net /~IO1 renamed /~{IO1}
- net /~IO2 renamed /~{IO2}
- net /~IRQ renamed /~{IRQ}
- net /~LED renamed /~{LED}
- net /~NMI renamed /~{NMI}
- net /~RESET renamed /~{RESET}
- net /~ROMH renamed /~{ROMH}
- net /~ROML renamed /~{ROML}
- net /~RST renamed /~{RST}
- net /~RST_O renamed /~{RST_O}
Other:
- net class Default removed
- net class power removed
